Commit message: Jazzy updates for baseline rviz

File: harvest_hardware/harvest_hardware_description/urdf/amiga_ur_gripper.urdf.xacro (robot description, xacro)
@@ -50,4 +50,5 @@
   <xacro:include filename="$(find harvest_hardware_description)/urdf/amiga.urdf.xacro"/>
   <xacro:include filename="$(find ur_description)/urdf/ur_macro.xacro"/>
+  <xacro:include filename="$(find ur_robot_driver)/urdf/ur.ros2_control.xacro"/>
   <xacro:include filename="$(find harvest_hardware_description)/urdf/finray_gripper.urdf.xacro"/>
   <xacro:include filename="$(find harvest_hardware_description)/urdf/gripper.urdf.xacro"/>
@@ -66,12 +67,18 @@
       physical_parameters_file   ="$(find ur_description)/config/$(arg ur_type)/physical_parameters.yaml"
       visual_parameters_file     ="$(find ur_description)/config/$(arg ur_type)/visual_parameters.yaml"
-      transmission_hw_interface="$(arg transmission_hw_interface)"
       safety_limits="$(arg safety_limits)"
       safety_pos_margin="$(arg safety_pos_margin)"
-      safety_k_position="$(arg safety_k_position)"
-      use_fake_hardware="$(arg use_fake_hardware)"
-      fake_sensor_commands="$(arg fake_sensor_commands)"
-      sim_gazebo ="$(arg sim_gazebo)"
-      sim_ignition ="$(arg sim_ignition)"
+      safety_k_position="$(arg safety_k_position)">
+    <origin xyz="0 0 0" rpy="0 0 0"/>
+  </xacro:ur_robot>
+  <!-- UR ros2_control -->
+  <xacro:ur_ros2_control
+      name="$(arg name)"
+      tf_prefix="$(arg tf_prefix)"
+      kinematics_parameters_file="$(find ur_description)/config/$(arg ur_type)/default_kinematics.yaml"
+      ur_type="$(arg ur_type)"
+      transmission_hw_interface="$(arg transmission_hw_interface)"
+      use_mock_hardware="$(arg use_fake_hardware)"
+      mock_sensor_commands="$(arg fake_sensor_commands)"
       headless_mode="$(arg headless_mode)"
       initial_positions="${xacro.load_yaml(initial_positions_file)}"
@@ -93,7 +100,5 @@
       reverse_port="$(arg reverse_port)"
       script_sender_port="$(arg script_sender_port)"
-      trajectory_port="$(arg trajectory_port)">
-    <origin xyz="0 0 0" rpy="0 0 0"/>
-  </xacro:ur_robot>
+      trajectory_port="$(arg trajectory_port)"/>
   <!-- mount finray gripper -->
   <xacro:if value="${gripper_type == 'finray'}">
